File: doc/PRU-BOARD-ST/untitled.kicad_sch (KiCad schematic)
At the start: 25 parts, among them J12 Program, J14 Conn_02x20_Odd_Even, J15 Conn_02x07_Odd_Even, J16 LED RGB, U1 ULN2003, U10 STM32F103C6Tx, U2 ULN2003, U9 AMS1117-3.3, Y2 12MHz

Commit message: 02-2026 - update
Connections:
- net SERVER-ON: now reaches U2.11 (O6)
Changed lines of the file:
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@@
 (kicad_sch
-	(version 20240812)
+	(version 20250114)
 	(generator "eeschema")
-	(generator_version "8.99")
+	(generator_version "9.0")
 	(paper "A4")
 	(text "GND pin 35 - 47"
@@
 	(wire
 		(pts
-			(xy 252.73 114.3) (xy 255.27 114.3)
+			(xy 252.73 114.3) (xy 257.81 114.3)
 		)
 		(stroke
@@
 			(effects
 				(font
+					(size 1.27 1.27)
+				)
+				(justify left)
+				(hide yes)
+			)
+		)
+	)
+	(global_label "SERVER-ON"
+		(shape output)
+		(at 257.81 114.3 0)
+		(fields_autoplaced yes)
+		(effects
+			(font
+				(size 1.27 1.27)
+			)
+			(justify left)
+		)
+		(property "Intersheetrefs" "${INTERSHEET_REFS}"
+			(at 272.1647 114.3 0)
+			(effects
+				(font
