File: doc/Tornio-Sch/Tornio/cpu.kicad_sch (KiCad schematic)
At the start: 0 parts

Commit message: spindle protection
Other:
- note removed: "CONTROL AXIS X"
- note removed: "CONTROL AXIS Y"
- note removed: "CONTROL AXIS Z"
- note removed: "CONTROL SPENDLE"
- note removed: "ETH"
- note removed: "LED BLUE"
- note removed: "LED RED"
- note removed: "LED YELLOW"
- note removed: "RPI 4"
- note removed: "SPI"
- note removed: "power 5Vdc"
Changed lines of the file:
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@@
 (kicad_sch
-	(version 20240812)
+	(version 20250114)
 	(generator "eeschema")
-	(generator_version "8.99")
+	(generator_version "9.0")
 	(paper "A4")
-	(rectangle
-		(start 82.55 63.5)
-		(end 196.85 100.33)
-		(stroke
-			(width 0)
-			(type default)
-		)
-		(fill
-			(type none)
-		)
-	)
-	(rectangle
-		(start 210.82 62.23)
-		(end 254 100.33)
-		(stroke
-			(width 0)
-			(type default)
-		)
-		(fill
-			(type none)
-		)
-	)
-	(text "ETH"
-		(exclude_from_sim no)
-		(at 221.742 40.894 0)
-		(effects
-			(font
-				(size 3.81 3.81)
-			)
-		)
-	)
-	(text "CONTROL AXIS X"
-		(exclude_from_sim no)
-		(at 91.694 85.852 0)
-		(effects
-			(font
-				(size 1.27 1.27)
-			)
-		)
-	)
-	(text "CONTROL AXIS Y"
-		(exclude_from_sim no)
-		(at 91.694 89.916 0)
-		(effects
-			(font
-				(size 1.27 1.27)
-			)
-		)
-	)
-	(text "power 5Vdc"
-		(exclude_from_sim no)
-		(at 226.568 22.86 0)
-		(effects
-			(font
-				(size 3.81 3.81)
-			)
-		)
-	)
-	(text "LED YELLOW"
-		(exclude_from_sim no)
-		(at 142.24 97.79 0)
-		(effects
-			(font
-				(size 1.27 1.27)
-			)
-		)
-	)
-	(text "LED BLUE"
-		(exclude_from_sim no)
-		(at 156.718 98.044 0)
-		(effects
-			(font
-				(size 1.27 1.27)
-			)
-		)
-	)
-	(text "LED RED"
-		(exclude_from_sim no)
-		(at 128.016 97.79 0)
-		(effects
-			(font
-				(size 1.27 1.27)
-			)
-		)
-	)
-	(text "SPI\n"
-		(exclude_from_sim no)
-		(at 204.724 88.646 0)
-		(effects
-			(font
-				(size 3.81 3.81)
-			)
-		)
-	)
-	(text "CONTROL AXIS Z"
-		(exclude_from_sim no)
-		(at 91.694 81.534 0)
-		(effects
-			(font
-				(size 1.27 1.27)
-			)
-		)
-	)
-	(text "RPI 4"
-		(exclude_from_sim no)
-		(at 232.156 69.596 0)
-		(effects
-			(font
-				(size 3.81 3.81)
-			)
-		)
-	)
-	(text "CONTROL SPENDLE"
-		(exclude_from_sim no)
-		(at 92.71 71.12 0)
-		(effects
-			(font
-				(size 1.27 1.27)
-			)
-		)
-	)
-	(bus
-		(pts
-			(xy 245.11 62.23) (xy 245.11 44.45)
-		)
-		(stroke
-			(width 0)
-			(type default)
-		)
-	)
-	(bus
-		(pts
-			(xy 71.12 71.12) (xy 82.55 71.12)
-		)
-		(stroke
-			(width 0)
-			(type default)
-		)
-	)
-	(bus
-		(pts
-			(xy 210.82 91.44) (xy 210.82 92.71)
-		)
-		(stroke
-			(width 0)
-			(type default)
-		)
-	)
-	(bus
-		(pts
-			(xy 196.85 91.44) (xy 210.82 91.44)
-		)
-		(stroke
-			(width 0)
-			(type default)
-		)
-	)
-	(bus
-		(pts
-			(xy 71.2576 82.55) (xy 82.6876 82.55)
-		)
-		(stroke
-			(width 0)
-			(type default)
-		)
-	)
-	(bus
-		(pts
-			(xy 71.12 86.36) (xy 82.55 86.36)
-		)
-		(stroke
-			(width 0)
-			(type default)
-		)
-	)
-	(bus
-		(pts
-			(xy 209.55 26.67) (xy 250.19 26.67)
-		)
-		(stroke
-			(width 0)
-			(type default)
-		)
-	)
-	(bus
-		(pts
-			(xy 71.12 90.17) (xy 82.55 90.17)
-		)
-		(stroke
-			(width 0)
-			(type default)
-		)
-	)
-	(bus
-		(pts
-			(xy 250.19 26.67) (xy 250.19 62.23)
-		)
-		(stroke
-			(width 0)
-			(type default)
-		)
-	)
-	(bus
-		(pts
-			(xy 213.36 44.45) (xy 245.11 44.45)
-		)
-		(stroke
-			(width 0)
-			(type default)
-		)
-	)
 )

Commit message: accessori
Parts:
- added C10, C12: 18p, symbol Device:C
- added C11: 47u, symbol Device:C_Polarized
- added C13, C14, C15, C16, C9: 100n, symbol Device:C
- added D5: V, Package_TO_SOT_THT:TO-18-2_Window, symbol LED:SFH460
- added D5: R, Package_TO_SOT_THT:TO-18-2_Window, symbol LED:SFH460
- added D6: G, Package_TO_SOT_THT:TO-18-2_Window, symbol LED:SFH460
- added J3: Program, symbol Connector_Generic:Conn_01x06
- added J5: Conn_02x20_Odd_Even, symbol Connector_Generic:Conn_02x20_Odd_Even
- added J7: Conn_02x07_Odd_Even, symbol Connector_Generic:Conn_02x07_Odd_Even
- added R14, R15: 10K, symbol Device:R
- added R16, R17, R18: 470, symbol Device:R
- added U10: STM32F103C6Tx, Package_QFP:LQFP-48_7x7mm_P0.5mm, symbol MCU_ST_STM32F1:STM32F103C6Tx
- added U2 (x2): ULN2003, symbol Transistor_Array:ULN2003
- added U9: AMS1117-3.3, Package_TO_SOT_SMD:SOT-223-3_TabPin2, symbol Regulator_Linear:AMS1117-3.3
- added Y2: 12MHz, symbol Device:Crystal
Connections:
- new net: D5.2 (A), R17.2
- new net: D5.2 (A), R16.2
- new net: R15.2, U10.44 (BOOT0)
- new net: C10.1, U10.5 (PD0), Y2.1
- new net: C12.1, U10.6 (PD1), Y2.2
- new net: D6.2 (A), R18.2
- new net ADC1: J7.4 (Pin_4), U10.18 (PB0)
- new net ADC2: J7.2 (Pin_2), U10.19 (PB1)
- new net D11_P-V-SpindleCPU: U10.43 (PB7)
- new net DIRA: U10.41 (PB5), U2.4 (I4)
- new net DIRA_5: U2.13 (O4)
- new net DIRX: U10.14 (PA4), U2.1 (I1)
- new net DIRX_5: U2.16 (O1)
- new net DIRY: U10.16 (PA6), U2.4 (I4)
- new net DIRY_5: U2.13 (O4)
- new net DIRZ: U10.15 (PA5), U2.1 (I1)
- new net DIRZ_5: U2.16 (O1)
- new net D_10-out-ex-loadcell: U10.40 (PB4)
- new net D_12-out-ex-uart: U10.42 (PB6)
- new net D_13-ex-i2c: U10.45 (PB8)
- new net D_14-ex-i2c: U10.46 (PB9)
- new net D_5: J7.6 (Pin_6), U10.30 (PA9)
- new net D_6: J7.8 (Pin_8), U10.31 (PA10)
- new net D_7: J7.7 (Pin_7), U10.33 (PA12)
- new net D_8-LEDV: R16.1, U10.38 (PA15)
- new net D_9: J7.9 (Pin_9)
- new net D_9-out-ex-loadcell: U10.39 (PB3), U2.6 (I6)
- new net ENC_CLK: J7.5 (Pin_5), U10.4 (PC15)
- new net ENC_DT: J7.3 (Pin_3), U10.3 (PC14)
- new net EN_AXIS_5: U2.14 (O3)
- new net FC_1: U10.20 (PB2)
- new net FC_2: U10.21 (PB10)
- new net FC_3: U10.22 (PB11)
- new net FC_4: U10.32 (PA11)
- new net GND: C10.2, C11.2, C12.2, C13.2, C14.2, C15.2, C16.2, C9.2, D5.1 (K), D6.1 (K), J3.1 (Pin_1), J5.14 (Pin_14), J5.20 (Pin_20), J5.30 (Pin_30), J5.34 (Pin_34), J5.39 (Pin_39), J5.6 (Pin_6), J5.9 (Pin_9), J7.13 (Pin_13), R15.1, U10.23 (VSS), U10.35 (VSS), U10.47 (VSS), U10.8 (VSSA), U2.8 (GND), U2.8 (GND), U9.1 (GND)
- new net NRST: J3.6 (Pin_6), R14.2, U10.7 (NRST)
- new net PWM SPINDLE: U10.29 (PA8), U2.7 (I7)
- new net PWM SPINDLE_5: U2.10 (O7)
- new net RGB-LED_5: U2.10 (O7)
- new net RGBLED: U10.17 (PA7), U2.7 (I7)
- new net SERVO-ON_5: U2.11 (O6)
- new net SPI2_CLK: J5.23 (Pin_23), U10.26 (PB13)
- new net SPI2_MISO: J5.21 (Pin_21), U10.27 (PB14)
- new net SPI2_MOSI: J5.19 (Pin_19), U10.28 (PB15)
- new net SPI2_NSS: J5.24 (Pin_24), U10.25 (PB12)
- new net STEPA: U10.13 (PA3), U2.5 (I5)
- new net STEPA_5: U2.12 (O5)
- new net STEPX: U10.10 (PA0), U2.2 (I2)
- new net STEPX_5: U2.15 (O2)
- new net STEPY: U10.11 (PA1), U2.5 (I5)
- new net STEPY_5: U2.12 (O5)
- new net STEPZ: U10.12 (PA2), U2.2 (I2)
- new net STEPZ_5: U2.15 (O2)
- new net SWCLK: J3.5 (Pin_5), U10.37 (PA14)
- new net SWDIO: J3.4 (Pin_4), U10.34 (PA13)
- new net SWO: J3.3 (Pin_3)
- new net V3_3: C11.1, C13.1, C14.1, C15.1, C16.1, C9.1, J3.2 (Pin_2), J7.1 (Pin_1), R14.1, R17.1, R18.1, U10.24 (VDD), U10.36 (VDD), U10.48 (VDD), U10.9 (VDDA), U9.2 (VO)
- new net V5: J5.2 (Pin_2), J5.4 (Pin_4), U2.9 (COM), U2.9 (COM), U9.3 (VI)
- new net _EN-AXIS: D5.1 (K), U10.2 (PC13), U2.3 (I3)
- no-connect marks 0 -> 1
Other:
- note added: "ATTIVO BASSO"
- note added: "BUS CPU"
- note added: "D11_P-V-SpindleCPU"
- note added: "D_9-out-ex-loadcell -> SERVO-ON_5"
- note added: "FC_1 -> asse X"
- note added: "GND pin 35 - 47"
