File: doc/Tornio-Sch/Tornio/Rimbalzo-Segnali.kicad_sch (KiCad schematic)
At the start: 10 parts, among them J1 Conn_02x25 INVERTER SANYO, J11 Screw_Terminal_01x12, J3 Screw_Terminal_01x12, J5 Screw_Terminal_01x10, J7 Screw_Terminal_01x16, J8 Conn_01x04, J9 Conn_02x08_Odd_Even, K1 Relay_DPDT

Commit message: accessori
Parts:
- removed J1: Conn_02x25 INVERTER SANYO, symbol Connector_Generic:Conn_02x25_Top_Bottom
- removed J11, J3: Screw_Terminal_01x12, symbol Connector:Screw_Terminal_01x12
- removed J5: Screw_Terminal_01x10, symbol Connector:Screw_Terminal_01x10
- removed J7: Screw_Terminal_01x16, symbol Connector:Screw_Terminal_01x16
- removed J8: Conn_01x04, symbol Connector_Generic:Conn_01x04
- removed R5: 10K, symbol Device:R
- added J12: Conn_02x08_Odd_Even, symbol Connector_Generic:Conn_02x08_Odd_Even
- added J13: Conn_02x12_Odd_Even, symbol Connector_Generic:Conn_02x12_Odd_Even
- added J14: Conn_01x06, symbol Connector_Generic:Conn_01x06
- added J9: FC, symbol Connector_Generic:Conn_01x06
- renumbered J9 to J?, K1 to K?
Connections:
- net +v12 is gone; now on net +V12: J?.10 (Pin_10)
- net +V12: now also J12.16 (Pin_16), J13.24 (Pin_24), J14.1 (Pin_1), J9.1 (Pin_1)
- net -V5: now also J12.14 (Pin_14), J14.5 (Pin_5)
- net ANA-SPINDLE: now also J13.21 (Pin_21)
- net ANA-SPINDLE-CPU: now also J12.11 (Pin_11)
- net COM-POWER- OUTPUT: now also J13.3 (Pin_3)
- net CONT2: now also J13.8 (Pin_8)
- net CONT3: now also J13.10 (Pin_10)
- net CONT5: now also J13.14 (Pin_14)
- net DIR-SPINDLE: now also J12.7 (Pin_7), J13.22 (Pin_22)
- net GND: now also J14.2 (Pin_2), J14.4 (Pin_4), J14.6 (Pin_6)
- net GND-ANA: now also J13.1 (Pin_1)
- net GND-CONT: now also J13.4 (Pin_4)
- net GND-Ext: now also J12.1 (Pin_1)
- net MON1: now also J13.23 (Pin_23)
- net OUT1: now also J13.5 (Pin_5)
- net OUT2: now also J13.7 (Pin_7)
- net OUT3: now also J13.9 (Pin_9)
- net OUT4: now also J13.11 (Pin_11)
- net OUT5: now also J13.13 (Pin_13)
- net PULS-SPINDLE: now also J12.5 (Pin_5), J13.20 (Pin_20)
- net SG: now also J13.16 (Pin_16)
- net SG-GND - F-PC / R-PC / ANA SPEED: now also J13.18 (Pin_18)
- net MANU / AUTO renamed SPINDLE AUTO_MANU
- net SERVO-AUTO-ON renamed SPINDLE ON CPU
- net SPINDLE ON CPU: now also J12.3 (Pin_3)
- net SERVO-ON renamed SPINDLE ON-OFF
- net SPINDLE ON-OFF: now also J13.6 (Pin_6)
- net SERVO-PANEL-ON renamed SPINDLE ON  PANEL
- net led-rgb renamed RGB-LED
- net RGB-LED: now also J12.15 (Pin_15)
- new net: J12.2 (Pin_2), J9.3 (Pin_3)
- new net: J12.4 (Pin_4), J9.4 (Pin_4)
- new net: J12.6 (Pin_6), J9.5 (Pin_5)
- new net: J12.8 (Pin_8), J9.6 (Pin_6)
- new net +V24: J14.3 (Pin_3)
- new net OUT6: J13.15 (Pin_15)
- new net SPINDLE MODE VELOCITY-POSITION : J12.9 (Pin_9), J13.12 (Pin_12)
Other:
- note added: "COMMAND PANEL"
- note added: "CPU - BOARD"
- note added: "FC - AXES"
- note added: "FC AXIS A"
- note added: "FC AXIS X"
- note added: "FC AXIS Y"
- note added: "FC AXIS Z"
- note added: "SERVO SPINDLE"
- note removed: "CPU"
- moved on the sheet: J?, K?, R6

Commit message: gg
Parts:
- added D7: 1N4007, Diode_THT:D_DO-41_SOD81_P10.16mm_Horizontal, symbol Diode:1N4007
- added J15: Conn_02x25 INVERTER SANYO, symbol Connector_Generic:Conn_02x25_Top_Bottom
Connections:
- net CONT2: now also J15.36 (Pin_36)
- net CONT3: now also J15.35 (Pin_35)
- net CONT5: now also J15.33 (Pin_33)
- net GND: now also J15.20 (Pin_20)
- net MON1: now also J15.30 (Pin_30)
- net OUT1: now also J15.39 (Pin_39)
- net OUT2: now also J15.40 (Pin_40)
- net OUT3: now also J15.41 (Pin_41)
- net OUT4: now also J15.42 (Pin_42)
- net SG: now also J15.31 (Pin_31)
- net SPINDLE MODE VELOCITY-POSITION : now also D7.2 (A)
- net SPINDLE ON  PANEL: now also D7.1 (K)
- net GND-CONT renamed SG GND
- new net CONT1: J15.37 (Pin_37)
- new net CONT4: J15.34 (Pin_34)
- new net F-PC-DIR: J15.26 (Pin_26)
- new net IN-COM: J15.50 (Pin_50)
- new net OUT-COM-PWR: J15.49 (Pin_49)
- new net R-PC-PULS: J15.28 (Pin_28)
- new net SG -GND-CONT: J15.38 (Pin_38)
- new net SG-GND: J15.47 (Pin_47), J15.48 (Pin_48)
- new net V-REF/T-REF: J15.21 (Pin_21)
Other:
- note added: "Ingressi attivi bassi (com +12V)"
- note added: "basso attivo Inverter"
