File: doc/Tornio-Sch/Tornio/Rimbalzo-Segnali.kicad_sch (KiCad schematic)
At the start: 9 parts, among them J12 Conn_02x08_Odd_Even, J13 Conn_02x12_Odd_Even, J14 Conn_01x06, J15 Conn_02x25 INVERTER SANYO, J9 FC

Commit message: eliminati file tenda da sole da accessori
Parts:
- added D8, D9: verde, symbol Device:LED
- added J16, J17: Axis X, symbol Connector_Generic:Conn_01x04
- added J18: Jumper, symbol Connector_Generic:Conn_02x04_Odd_Even
- added K1, K2: Relay_DPDT, symbol Relay:Relay_DPDT
- added Q1: BC327, Package_TO_SOT_THT:TO-92_Inline, symbol Transistor_BJT:BC327
- added R23, R7: 1k2, symbol Device:R
- added R24: 4k7, symbol Device:R
Connections:
- net +V12: now also D8.2 (A), D9.2 (A), K1.A1, K2.A1, Q1.3 (E)
- net GND: no longer J15.20 (Pin_20)
- net OUT3: no longer J13.9 (Pin_9)
- net SPINDLE AUTO_MANU: now also D7.2 (A), J13.12 (Pin_12); no longer K?.A2
- net SPINDLE MODE VELOCITY-POSITION : now also D7.1 (K), K?.A2; no longer D7.2 (A), J13.12 (Pin_12)
- net SPINDLE ON  PANEL: no longer D7.1 (K)
- net D12-OUT: now reaches J12.10 (Pin_10)
- net D12-OUT: now also K2.A2, R23.1
- net D10-OUT-COOL_5: now reaches J12.12 (Pin_12)
- net D10-OUT-COOL_5: now also K1.A2, R7.1
- net at J12.8 (Pin_8), J9.6 (Pin_6): now also Q1.1 (C)
- net gnd SG-39-46 (pin 24-24 servo): now reaches J13.19 (Pin_19)
- net ZOP Zero Encoder Pos: now reaches J15.11 (Pin_11)
- net ZOP Zero Encoder Pos: now also J18.7 (Pin_7), R24.1
- net SG pin 3-11  : now reaches J15.12 (Pin_12)
- net Out A phase Encoder: now reaches J15.3 (Pin_3)
- net Out A phase Encoder: now also J18.1 (Pin_1)
- net _Out A phase Encoder: now reaches J15.4 (Pin_4)
- net _Out A phase Encoder: now also J18.2 (Pin_2)
- net Out B phase Encoder: now reaches J15.5 (Pin_5)
- net Out B phase Encoder: now also J18.3 (Pin_3)
- net _Out B phase Encoder: now reaches J15.6 (Pin_6)
- net _Out B phase Encoder: now also J18.4 (Pin_4)
- net Out Z phase Encoder: now reaches J15.7 (Pin_7)
- net Out Z phase Encoder: now also J18.5 (Pin_5)
- net _Out Z phase Encoder: now reaches J15.8 (Pin_8)
- net _Out Z phase Encoder: now also J18.6 (Pin_6)
- net DIR-SPINDLE renamed DIR_A-SPINDLE
- net LED verde renamed __SPINDLE-ON-LED
- net __SPINDLE-ON-LED: now also J13.9 (Pin_9)
- net PULS-SPINDLE renamed PULS_A-SPINDLE
- new net: J17.4 (Pin_4), K1.21
- new net: J17.1 (Pin_1), K1.22
- new net: J17.2 (Pin_2), K1.24
- new net: Q1.2 (B), R24.2
- new net: D9.1 (K), R23.2
- new net: J16.4 (Pin_4), K2.21
- new net: J16.1 (Pin_1), K2.22
- new net: J16.2 (Pin_2), K2.24
- new net: D8.1 (K), R7.2
- new net SG pin 3-11: J18.8 (Pin_8)
Other:
- note added: "ENCODER SANYO"
- note added: "ENCODER SPINDLE"
- note added: "FC AXIS A IN 3"
- note added: "FC AXIS X IN 0"
- note added: "FC AXIS Y IN 1"
- note added: "FC AXIS Z IN 2"
- note added: "basso analogico alto impulsi"
- note removed: "FC AXIS A"
- note removed: "FC AXIS X"
- note removed: "FC AXIS Y"
- note removed: "FC AXIS Z"
- moved on the sheet: D7, J12, J14, J15, J9
