File: doc/Tornio-Sch/Tornio/panel.sch.kicad_sch (KiCad schematic)
At the start: 18 parts, among them J10 Conn_01x04, J2 Conn_02x08_Odd_Even, J4 sensore hall, J6 display, SW1 CW / CCW, SW12 SPINDLE MANU / AUTO, SW2 XXXX, SW8 SPINDLE ON/OFF, U1 L7805

Commit message: accessori
Other:
- note added: "1° da SX"
- note added: "2°"
- note added: "3°"
- note added: "4°"
- note removed: "1 da SX"
- note removed: "2"
- note removed: "3"
- note removed: "4"
Changed lines of the file:
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@@
 		)
 	)
-	(text "3\n"
+	(text "3°\n"
 		(exclude_from_sim no)
 		(at 150.876 37.846 0)
@@
 		)
 	)
-	(text "2"
+	(text "2°"
 		(exclude_from_sim no)
 		(at 136.906 37.846 0)
@@
 		)
 	)
-	(text "4\n"
+	(text "4°\n"
 		(exclude_from_sim no)
 		(at 161.544 37.338 0)
@@
 		)
 	)
-	(text "1 da SX"
+	(text "1° da SX"
 		(exclude_from_sim no)
 		(at 183.134 80.01 0)

Commit message: gg
Other:
- note added: "1 - NERO"
- note added: "10 - AZZURRO"
- note added: "11 - BIANCO DEL GIALLO SCURO"
- note added: "12 - ARANCIO"
- note added: "13 - VERDE"
- note added: "14 - ROSSO"
- note added: "15 - BIANCO DEL VERDE"
- note added: "2 - BIANCO DA SOLO"
- note added: "3 -"
- note added: "4 - BIANCO"
- note added: "5 - VIOVA CHIARO"
- note added: "6 - MARRONE CHIARO"
- note added: "7 - BIANCO DEL VIOLA"
- note added: "8 - BIANCO DEL MARRONE CHIARO"
- note added: "9 - GIALLO SCURO"
Changed lines of the file:
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@@
+		)
+	)
+	(text "12 - ARANCIO"
+		(exclude_from_sim no)
+		(at 20.066 82.042 0)
+		(effects
+			(font
+				(size 1.27 1.27)
+			)
 		)
 	)
@@
 	(text "(BIANCO) ON/OFF"
 		(exclude_from_sim no)
-		(at 30.988 62.992 0)
+		(at -26.416 62.992 0)
+		(effects
+			(font
+				(size 1.27 1.27)
+			)
+		)
+	)
+	(text "5 - VIOVA CHIARO"
+		(exclude_from_sim no)
+		(at 23.114 67.564 0)
 		(effects
 			(font
@@
 	(text "DIR"
 		(exclude_from_sim no)
-		(at 29.464 72.898 0)
+		(at -27.94 72.898 0)
 		(effects
 			(font
@@
 		)
 	)
+	(text "14 - ROSSO"
+		(exclude_from_sim no)
+		(at 19.304 85.852 0)
+		(effects
+			(font
+				(size 1.27 1.27)
+			)
+		)
+	)
+	(text "1 - NERO"
+		(exclude_from_sim no)
+		(at 19.304 59.69 0)
+		(effects
+			(font
+				(size 1.27 1.27)
+			)
+		)
+	)
+	(text "15 - BIANCO DEL VERDE"
+		(exclude_from_sim no)
+		(at 25.146 87.884 0)
+		(effects
+			(font
+				(size 1.27 1.27)
+			)
+		)
+	)
 	(text "(ARANCIO) ANA SPEED (0-10V)\n"
 		(exclude_from_sim no)
-		(at 37.338 58.166 0)
+		(at -20.066 58.166 0)
 		(effects
 			(font
@@
 		)
 	)
+	(text "9 - GIALLO SCURO"
+		(exclude_from_sim no)
+		(at 23.368 75.946 0)
+		(effects
+			(font
+				(size 1.27 1.27)
+			)
+		)
+	)
+	(text "13 - VERDE"
+		(exclude_from_sim no)
+		(at 19.05 84.074 0)
+		(effects
+			(font
+				(size 1.27 1.27)
+			)
+		)
+	)
+	(text "11 - BIANCO DEL GIALLO SCURO"
+		(exclude_from_sim no)
+		(at 28.956 80.01 0)
+		(effects
+			(font
+				(size 1.27 1.27)
+			)
+		)
+	)
 	(text "PULSE"
 		(exclude_from_sim no)
-		(at 30.734 71.374 0)
+		(at -26.67 71.374 0)
 		(effects
 			(font
@@
 	(text "(VERDE) ANA/PULSE"
 		(exclude_from_sim no)
-		(at 32.766 60.452 0)
+		(at -24.638 60.452 0)
+		(effects
+			(font
+				(size 1.27 1.27)
+			)
+		)
+	)
+	(text "7 - BIANCO DEL VIOLA"
+		(exclude_from_sim no)
+		(at 25.146 71.882 0)
 		(effects
 			(font
@@
 		)
 	)
+	(text "4 - BIANCO"
+		(exclude_from_sim no)
+		(at 20.066 65.786 0)
+		(effects
+			(font
+				(size 1.27 1.27)
+			)
+		)
+	)
+	(text "3 - "
+		(exclude_from_sim no)
+		(at 16.764 63.754 0)
+		(effects
+			(font
+				(size 1.27 1.27)
+			)
+		)
+	)
+	(text "2 - BIANCO DA SOLO "
+		(exclude_from_sim no)
+		(at 25.4 61.722 0)
+		(effects
+			(font
+				(size 1.27 1.27)
+			)
+		)
+	)
 	(text "-5"
 		(exclude_from_sim no)
-		(at 46.99 75.946 0)
+		(at -10.414 75.946 0)
+		(effects
+			(font
+				(size 1.27 1.27)
+			)
+		)
+	)
+	(text "6 - MARRONE CHIARO"
+		(exclude_from_sim no)
+		(at 24.892 69.596 0)
+		(effects
+			(font
+				(size 1.27 1.27)
+			)
+		)
+	)
+	(text "8 - BIANCO DEL MARRONE CHIARO"
+		(exclude_from_sim no)
+		(at 30.988 73.914 0)
+		(effects
+			(font
+				(size 1.27 1.27)
+			)
+		)
+	)
+	(text "10 - AZZURRO"
+		(exclude_from_sim no)
+		(at 20.32 77.978 0)
 		(effects
 			(font
@@
 	(text "+12Vcc"
 		(exclude_from_sim no)
-		(at 47.498 73.66 0)
-		(effects
-			(font
+		(at -9.906 73.66 0)
+		(effects
+			(font
