File: doc/Tornio-Sch/Tornio/panel.sch.kicad_sch (KiCad schematic)
At the start: 18 parts, among them J10 Conn_01x04, J2 Conn_02x08_Odd_Even, J4 sensore hall, J6 display, SW1 CW / CCW, SW12 SPINDLE MANU / AUTO, SW2 XXXX, SW8 SPINDLE ON/OFF, U1 L7805

Commit message: eliminati file tenda da sole da accessori
Connections:
- net K verde renamed _SPINDLE-ON
- net _SPINDLE-ON: no longer J2.14 (Pin_14)
- new net __SPINDLE-ON-LED: J2.14 (Pin_14)
Changed lines of the file:
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@@
 	(generator_version "9.0")
 	(paper "A4")
+	(title_block
+		(date "2026-07-28")
+		(rev "1.0")
+	)
 	(rectangle
 		(start 58.42 30.48)
@@
 	(wire
 		(pts
-			(xy 68.58 68.58) (xy 68.58 46.99)
+			(xy 66.04 68.58) (xy 66.04 46.99)
 		)
 		(stroke
@@
 	(wire
 		(pts
-			(xy 76.2 59.69) (xy 76.2 63.5)
+			(xy 72.39 55.88) (xy 72.39 63.5)
 		)
 		(stroke
@@
 	(wire
 		(pts
-			(xy 99.06 68.58) (xy 68.58 68.58)
+			(xy 99.06 68.58) (xy 66.04 68.58)
 		)
 		(stroke
@@
 	(wire
 		(pts
-			(xy 68.58 46.99) (xy 137.16 46.99)
-		)
-		(stroke
-			(width 0)
-			(type default)
-		)
-	)
-	(wire
-		(pts
-			(xy 76.2 63.5) (xy 99.06 63.5)
+			(xy 66.04 46.99) (xy 137.16 46.99)
+		)
+		(stroke
+			(width 0)
+			(type default)
+		)
+	)
+	(wire
+		(pts
+			(xy 72.39 63.5) (xy 99.06 63.5)
 		)
 		(stroke
@@
 		)
 	)
-	(global_label "K verde"
+	(global_label "__SPINDLE-ON-LED"
 		(shape input)
 		(at 97.79 58.42 180)
@@
 		)
 		(property "Intersheetrefs" "${INTERSHEET_REFS}"
-			(at 87.4872 58.42 0)
+			(at 75.7548 58.42 0)
 			(effects
 				(font
@@
 		)
 	)
-	(global_label "K verde"
+	(global_label "_SPINDLE-ON"
 		(shape input)
 		(at 201.93 134.62 180)
@@
 		)
 		(property "Intersheetrefs" "${INTERSHEET_REFS}"
-			(at 191.6272 134.62 0)
+			(at 185.8819 134.62 0)
 			(effects
 				(font
@@
 	(symbol
 		(lib_id "power:VCC")
-		(at 76.2 59.69 0)
+		(at 72.39 55.88 0)
 		(unit 1)
 		(exclude_from_sim no)
@@
 		(dnp no)
 		(property "Reference" "#PWR010"
-			(at 76.2 63.5 0)
+			(at 72.39 59.69 0)
 			(effects
 				(font
@@
 		)
 		(property "Value" "+V12"
-			(at 76.2 55.88 0)
+			(at 72.39 52.07 0)
 			(effects
 				(font
@@
 		)
 		(property "Footprint" ""
-			(at 76.2 59.69 0)
+			(at 72.39 55.88 0)
 			(effects
 				(font
@@
 		)
 		(property "Datasheet" ""
-			(at 76.2 59.69 0)
+			(at 72.39 55.88 0)
 			(effects
 				(font
@@
 		)
 		(property "Description" "Power symbol creates a global label with name \"VCC\""
-			(at 76.2 59.69 0)
-			(effects
-				(font
+			(at 72.39 55.88 0)
+			(effects
+				(font
