File: doc/Tornio-Sch/Tornio/Tornio.kicad_sch (KiCad schematic)
At the start: 0 parts

Commit message: eliminati file tenda da sole da accessori
Other:
- note added: "LAYOUT ELECTRICAL CABINET"
- note added: "POWER"
- note added: "SUPPLY"
