File: doc/Tornio-Sch/Tornio/cpu-2_sch.kicad_sch (KiCad schematic)
At the start: 31 parts, among them J1 Conn_02x08_Odd_Even, J11 Axis X, J19 Axis Y, J20 Axis Z, J8 Jumper, U11 HCPL-0630, U12 LM2904, U3 HCPL-0630, U5 LTV-817, U6 LTV-817, U7 LTV-817, U8 LTV-817

Commit message: eliminati file tenda da sole da accessori
Parts:
- added U4: TC4422, Package_DIP:DIP-8_W7.62mm, symbol Driver_FET:TC4422
- R11, R12, R13, R19: value 470 -> 1K2
- R27: value 56k -> 5K6
- U12: value LM2904 -> LM833
Connections:
- net DIRX_5: now also J11.2 (Pin_2); no longer J11.1 (Pin_1)
- net DIRY_5: now also J19.2 (Pin_2); no longer J19.1 (Pin_1)
- net DIRZ_5: now also J20.2 (Pin_2); no longer J20.1 (Pin_1)
- net EN_AXIS_5: now also J11.1 (Pin_1), J19.1 (Pin_1), J20.1 (Pin_1); no longer J11.3 (Pin_3), J19.3 (Pin_3), J20.3 (Pin_3)
- net STEPX_5: now also J11.3 (Pin_3); no longer J11.2 (Pin_2)
- net STEPY_5: now also J19.3 (Pin_3); no longer J19.2 (Pin_2)
- net STEPZ_5: now also J20.3 (Pin_3); no longer J20.2 (Pin_2)
- net at R10.1, R22.1: now also U4.6 (OUTPUT), U4.7 (OUTPUT); no longer U3.7 (VO1)
- net D12-OUT: now reaches J1.10 (Pin_10)
- net D10-OUT-COOL_5: now reaches J1.12 (Pin_12)
- net at U3.6 (VO2): no longer J1.9 (Pin_9)
- net SERVO-ON_5 renamed D9-SERVO-ON_5
- new net: U4.1 (VDD), U4.8 (VDD)
- new net: U4.4 (GND), U4.5 (GND)
- new net D11-P-V-OUT_5: J1.9 (Pin_9)
- new net PWM SPINDLE: U4.2 (INPUT)
Other:
- note added: "10 - GIALLO"
- note added: "12 - GRIGIO"
- note added: "14 - ARANCIO/GRIGIO"
- note added: "16 - BIANCO"
- note added: "2 - ARANCIO"
- note added: "4 - BLU"
- note added: "6 - ROSA"
- note added: "8 - AZZURRO"
- note added: "CALZA - 1"
- note added: "CAVO 15 + CALZA"
- note added: "GIALLO/ROSSO - 15"
- note added: "MARRONE - 7"
- note added: "MARRONE/VERDE - 11"
- note added: "NERO - 5"
- note added: "ROSSO - 13"
- note added: "VERDE - 3"
- note added: "VIOLA - 9"
- moved on the sheet: R8, R9, U3
