File: doc/Tornio-Sch/Tornio/servo-motor.kicad_sch (KiCad schematic)
At the start: 0 parts

Commit message: eliminati file tenda da sole da accessori
Parts:
- added SW3: Zero Z, symbol Switch:SW_Push_SPDT
- added SW4: Zero X, symbol Switch:SW_Push_SPDT
- added SW5: Zero Y, symbol Switch:SW_Push_SPDT
Other:
- note added: "1 - Nero +A 2 - Grigio +B 3 - Marrone -A 4 - giallo / Verde -B"
- note added: "AXIS Z VERTICAL"
- note added: "Connector 4 P"
- note added: "DIP="
- note added: "DIP=1010 00"
- note added: "DIR -> Orange"
- note added: "DM860H"
- note added: "EN -> Red"
- note added: "GND -> Black"
- note added: "HBS 860H"
- note added: "PULSE -> Green"
- note added: "STEPPER"
- note added: "WITH ENCODER 4000 STEP"
- note removed: "AXIS Y VERTICAL"
- note removed: "DIRECTION"
- note removed: "ENABLE"
- note removed: "PULSE"
